File: lippa.sch (EAGLE design)
At the start: 109 parts, among them K1 629105136821, X1 B4B-PH-K-S, X2 B4B-PH-K-S, X3 B4B-PH-K-S, X4 B4B-PH-K-S, X5 LIITTIMET_X3815-10, X8 PS-JOYSTICK, Y1 EKE_PTH3.2-6.5SQ, Y2 EKE_PTH3.2-6.5SQ, Y3 EKE_PTH3.2-6.5SQ, Y4 EKE_PTH3.2-6.5SQ

Commit message: wip
Parts:
- removed D1: STM32F407ZG, omat_ic_2:STM32F407ZG
- added D2: STM32F407VE, lippa:STM32F407VE
- added X6: (no value), lippa:TE_RUUVILIITIN2
Connections:
- removed net DIR_4: D1G$3.PE12
- removed net DIR_5: D1G$3.PE13
- removed net ENABLE_N: D1G$3.PE14
- removed net ENA_4: D1G$3.PG4
- removed net ENA_5: D1G$3.PG5
- removed net INPUT_0: D1G$2.PC8
- removed net INPUT_1: D1G$2.PC9
- removed net INPUT_10: D1G$2.PD2
- removed net INPUT_11: D1G$2.PD3
- removed net INPUT_12: D1G$2.PD4
- removed net INPUT_13: D1G$2.PD5
- removed net INPUT_14: D1G$2.PD6
- removed net INPUT_15: D1G$2.PD7
- removed net INPUT_2: D1G$2.PC10
- removed net INPUT_3: D1G$2.PC11
- removed net INPUT_4: D1G$2.PC12
- removed net INPUT_5: D1G$2.PC13
- removed net INPUT_8: D1G$2.PD0
- removed net INPUT_9: D1G$2.PD1
- removed net N$14: N1.NENBL/AENBL
- removed net N$15: N1.STEP/BENBL
- removed net N$16: N1.DIR/BPHASE
- removed net N$28: N2.NENBL/AENBL
- removed net N$29: N2.STEP/BENBL
- removed net N$30: N2.DIR/BPHASE
- removed net N$43: N3.NENBL/AENBL
- removed net N$44: N3.STEP/BENBL
- removed net N$45: N3.DIR/BPHASE
- removed net N$58: N4.NENBL/AENBL
- removed net N$59: N4.STEP/BENBL
- removed net N$60: N4.DIR/BPHASE
- removed net OUT_1: D1G$2.PC0
- removed net OUT_2: D1G$2.PC1
- removed net OUT_3: D1G$2.PB10
- removed net OUT_4: D1G$2.PB11
- removed net PULSE_4: D1G$2.PB8
- removed net PULSE_5: D1G$2.PB9
- removed net SERVO_PWM_3: D1G$2.PB0
- removed net SPARE_1: D1G$3.PG6
- removed net SPARE_2: D1G$3.PG7
- new net PULSE_1: D2G$2.PC6, N2.STEP/BENBL
- net +3V3: now also D2G$1.VBAT, D2G$1.VDD1, D2G$1.VDD2, D2G$1.VDD3, D2G$1.VDD4, D2G$1.VDD5, D2G$1.VDD6; no longer D1G$1.PDR_ON, D1G$1.VBAT, D1G$1.VDD1, D1G$1.VDD10, D1G$1.VDD11, D1G$1.VDD12, D1G$1.VDD2, D1G$1.VDD3, D1G$1.VDD4, D1G$1.VDD5, D1G$1.VDD6, D1G$1.VDD7, D1G$1.VDD8, D1G$1.VDD9
- net +VBAT: now also X6.1
- net BOOT0: now also D2G$1.BOOT0; no longer D1G$1.BOOT0
- net DIR_0: now also D2G$3.PE8, N1.DIR/BPHASE; no longer D1G$3.PE8
- net DIR_1: now also D2G$3.PE10, N2.DIR/BPHASE; no longer D1G$3.PE9
- net DIR_2: now also D2G$3.PE11, N3.DIR/BPHASE; no longer D1G$3.PE10
- net DIR_3: now also D2G$3.PE12, N4.DIR/BPHASE; no longer D1G$3.PE11
- net ENABLE_PWM_N: now also D2G$2.PD4; no longer D1G$3.PG9
- net ENA_0: now also D2G$2.PD0, N1.NENBL/AENBL; no longer D1G$3.PG0
- net ENA_1: now also D2G$2.PD1, N2.NENBL/AENBL; no longer D1G$3.PG1
- net ENA_2: now also D2G$2.PD2, N3.NENBL/AENBL; no longer D1G$3.PG2
- net ENA_3: now also D2G$2.PD3, N4.NENBL/AENBL; no longer D1G$3.PG3
- net GND: now also D2G$1.VSS1, D2G$1.VSS2, D2G$1.VSS3, D2G$1.VSS4, D2G$1.VSSA, X6.2; no longer D1G$1.VSS1, D1G$1.VSS2, D1G$1.VSS3, D1G$1.VSS4, D1G$1.VSS5, D1G$1.VSS6, D1G$1.VSS7, D1G$1.VSS8, D1G$1.VSS9, D1G$1.VSSA
- net I2C1SCL: now also D2G$2.PB6; no longer D1G$2.PB6
- net I2C1SDA: now also D2G$2.PB7; no longer D1G$2.PB7
- net LED_DEBUG: now also D2G$2.PC2; no longer D1G$2.PC2
- net LED_ERR: now also D2G$2.PC4; no longer D1G$2.PC4
- net LED_RUN: now also D2G$2.PC3; no longer D1G$2.PC3
- net MEAS12V: now also D2G$1.PA0/WKUP; no longer D1G$1.PA0/WKUP
- net N$62: now also D2G$1.PB2/BOOT1; no longer D1G$1.PB2/BOOT1
- net N$63: now also D2G$1.PA14/TCK/SWCLK; no longer D1G$1.PA14/TCK/SWCLK
- net N$73: now also D2G$1.PA13/TMS/SWDIO; no longer D1G$1.PA13/TMS/SWDIO
- net OSCIN: now also D2G$1.PH0/OSCIN; no longer D1G$1.PH0/OSCIN
- net OSCOUT: now also D2G$1.PH1/OSCOUT; no longer D1G$1.PH1/OSCOUT
- net PULSE_0: now also D2G$2.PD12, N1.STEP/BENBL; no longer D1G$2.PD12
- net PULSE_2: now also D2G$3.PE5, N3.STEP/BENBL; no longer D1G$2.PC6
- net PULSE_3: now also D2G$2.PB8, N4.STEP/BENBL; no longer D1G$3.PE5
- net RESETL: now also D2G$1.RSTL; no longer D1G$1.RSTL
- net SERVO_PWM_1: now also D2G$2.PA6; no longer D1G$2.PA6
- net SERVO_PWM_2: now also D2G$2.PA7; no longer D1G$2.PA7
- net SPI1CLK: now also D2G$1.PB3/TDO; no longer D1G$1.PB3/TDO
- net SPI1MISO: now also D2G$1.PB4/TRSTL; no longer D1G$1.PB4/TRSTL
- net SPI1MOSI: now also D2G$2.PB5; no longer D1G$2.PB5
- net SPI_CS_PS2_N: now also D2G$2.PA1; no longer D1G$2.PA1
- net USART1RX: now also D2G$2.PA10; no longer D1G$2.PA10
- net USART1TX: now also D2G$2.PA9; no longer D1G$2.PA9
- net USART1TXE: now also D2G$2.PD15; no longer D1G$2.PD15
- net USART2TX: now also D2G$2.PA2; no longer D1G$2.PA2
- net USART3RX: now also D2G$2.PD9; no longer D1G$2.PD9
- net USART3TX: now also D2G$2.PD8; no longer D1G$2.PD8
- net USBRENUM: now also D2G$2.PB15; no longer D1G$2.PB15
- net USB_DM: now also D2G$2.PA11; no longer D1G$2.PA11
- net USB_DP: now also D2G$2.PA12; no longer D1G$2.PA12
- net VCAP1: now also D2G$1.VCAP1; no longer D1G$1.VCAP1
- net VCAP2: now also D2G$1.VCAP2; no longer D1G$1.VCAP2
- net VDDA: now also D2G$1.VDDA; no longer D1G$1.VDDA
- net VREF25: now also D2G$1.VREF+; no longer D1G$1.VREF+

Commit message: more wip
Parts:
- added C34, C35, C36, C37: (no value), lippa:OMAT_IC_2_CAP0603
- added C38, C42: 100n 0603, lippa:OMAT_IC_2_CAP0603
- added C39, C40, C41, C43, C44, C45, C49: 22u 25V, lippa:OMAT_IC_2_CAP0805
- added C46: 100n, omat_ic_2:CAP0603
- added C48: 2u2, omat_ic_2:CAP0603
- added D1: 74AHCT125, lippa:74AHCT125
- added L1: NRS4018-2U2, lippa:NRS4018-2U2
- added L4: NRS4018-4U7, lippa:NRS4018-4U7
- added L5: IND0603, omat_ic_2:IND0603
- added N6, N7: TPS561201, lippa:TPS561201
- added R40, R41, R42: (no value), lippa:OMAT_IC_2_RES0603
- added R43: 54k9, lippa:OMAT_IC_2_RES0603
- added R44, R46: 10k0, lippa:OMAT_IC_2_RES0603
- added R45: 33k2, lippa:OMAT_IC_2_RES0603
- added R47, R48: (no value), cpu:RES0603
- added R49, R50, R51, R52, R53: 2k00, omat_ic_2:RES0603
- added V2, V3, V4: SK34A, lippa:SK34A
- added V5: SMAJXXA, lippa:SMAJXXA
- added X10, X7, X9: PIIKKIRIMA-3, lippa:PIIKKIRIMA-3
- added X11: B8B-PH-K-S, lippa:B8B-PH-K-S
- X8: value PS-JOYSTICK -> B6B-PH-K-S; device cpu:PS-JOYSTICK -> lippa:B6B-PH-K-S
Connections:
- net MEAS12V renamed MEASVBAT
- net N$62 renamed BOOT1
- net N$63 renamed SWCLK_CPU
- net N$73 renamed SWDIO_CPU
- removed net DIR_0: D2G$3.PE8, N1.DIR/BPHASE
- removed net ENA_0: D2G$2.PD0, N1.NENBL/AENBL
- removed net ENA_1: D2G$2.PD1, N2.NENBL/AENBL
- removed net ENA_2: D2G$2.PD2, N3.NENBL/AENBL
- removed net ENA_3: D2G$2.PD3, N4.NENBL/AENBL
- removed net N$17: C6.1, N2.VINT
- removed net N$2: C2.1, N1.VINT
- removed net N$32: C10.1, N3.VINT
- removed net N$47: C14.1, N4.VINT
- removed net N$70: R86.1, X8.CMD
- removed net PULSE_0: D2G$2.PD12, N1.STEP/BENBL
- removed net USART2TX: D2G$2.PA2
- new net +5V: C34.1, C40.1, C41.1, D1.VCC, L4.1, L5.2, R43.2
- new net ATT: R87.1, X8.5
- new net CLK: R88.1, X8.6
- new net CMD: R86.1, X8.2
- new net DATA: R38.1, X8.1
- new net DIR_4: D2G$3.PE12, N4.DIR/BPHASE
- new net ENA_1_N: D2G$2.PD0, N1.NENBL/AENBL, R50.1
- new net ENA_2_N: D2G$2.PD1, N2.NENBL/AENBL, R51.1
- new net ENA_3_N: D2G$2.PD2, N3.NENBL/AENBL, R52.1
- new net ENA_4_N: D2G$2.PD3, N4.NENBL/AENBL, R53.1
- new net LIDAR_VCC: C46.1, C48.1, L5.1, X11.6, X11.8
- new net MODE_1: D2G$2.PC10, N1.M0/APHASE
- new net MODE_2: D2G$2.PC11, N2.M0/APHASE
- new net MODE_3: D2G$2.PC12, N3.M0/APHASE
- new net MODE_4: D2G$2.PC13, N4.M0/APHASE
- new net N$14: R41.2, X9.1
- new net N$15: R40.2, X7.1
- new net N$16: R42.2, X10.1
- new net N$28: D1.Y1, R40.1
- new net N$29: D1.Y2, R41.1
- new net N$30: D1.Y3, R42.1
- new net N$43: C38.1, L4.2, N6.SW
- new net N$44: C37.1, V4.C, X10.2
- new net N$45: C36.1, V3.C, X9.2
- new net N$58: C35.1, V2.C, X7.2
- new net N$59: C38.2, N6.BST
- new net N$60: N6.FB, R43.1, R44.2
- new net N$74: C42.1, L1.2, N7.SW
- new net N$75: C42.2, N7.BST
- new net N$76: N7.FB, R45.1, R46.2
- new net PULSE_4: D2G$2.PB8, N4.STEP/BENBL
- new net SERVO_PWM_3: D1.A3, D2G$2.PB0
- new net VINT_1: C2.1, N1.CONFIG, N1.M1, N1.VINT
- new net VINT_2: C6.1, N2.CONFIG, N2.M1, N2.VINT
- new net VINT_3: C10.1, N3.CONFIG, N3.M1, N3.VINT
- new net VINT_4: C14.1, N4.CONFIG, N4.M1, N4.VINT
- net +3V3: now also C44.1, C45.1, L1.1, R45.2, R49.2, R50.2, R51.2, R52.2, R53.2
- net +VBAT: now also C39.1, C43.1, C49.1, N6.ENA, N6.VIN, N7.ENA, N7.VIN, V2.A, V3.A, V4.A, V5.C
- net DIR_1: now also D2G$3.PE8, N1.DIR/BPHASE; no longer D2G$3.PE10, N2.DIR/BPHASE
- net DIR_2: now also D2G$3.PE10, N2.DIR/BPHASE; no longer D2G$3.PE11, N3.DIR/BPHASE
- net DIR_3: now also D2G$3.PE11, N3.DIR/BPHASE; no longer D2G$3.PE12, N4.DIR/BPHASE
- net ENABLE_PWM_N: now also D1.OE1, D1.OE2, D1.OE3, R49.1
- net FAULT_N: now also D2G$2.PD6
- net GND: now also C34.2, C35.2, C36.2, C37.2, C39.2, C40.2, C41.2, C43.2, C44.2, C45.2, C46.2, C48.2, C49.2, D1.A4, D1.GND, D1.OE4, N6.GND, N7.GND, R44.1, R46.1, V5.A, X10.3, X11.3, X7.3, X8.3, X9.3; no longer X8.GND
- net LED_DEBUG: now also D2G$3.PE2; no longer D2G$2.PC2
- net LED_ERR: now also D2G$3.PE4; no longer D2G$2.PC4
- net LED_RUN: now also D2G$3.PE3; no longer D2G$2.PC3
- net N$69: now also X11.4, X11.7; no longer R38.1, X8.DATA
- net N$71: now also R48.1, X11.2; no longer R87.1, X8.ATT
- net N$72: now also R47.1, X11.5; no longer R88.1, X8.CLK
- net PSVCC: now also X8.4; no longer X8.VCC
- net PULSE_1: now also D2G$2.PD12, N1.STEP/BENBL; no longer D2G$2.PC6, N2.STEP/BENBL
- net PULSE_2: now also D2G$2.PC6, N2.STEP/BENBL; no longer D2G$3.PE5, N3.STEP/BENBL
- net PULSE_3: now also D2G$3.PE5, N3.STEP/BENBL; no longer D2G$2.PB8, N4.STEP/BENBL
- net SERVO_PWM_1: now also D1.A1
- net SERVO_PWM_2: now also D1.A2
- net SLEEP_N: now also D2G$2.PD5
- net USART1RX: now also R47.2
- net USART1TX: now also R48.2
Other:
- note added: "INDEXER MODE (MODE_x) 0 : 8 microstep 1 : 16 microstep Z : 32 microstep"
- moved on the sheet: C10, C14, C2, C6, C61, C62, L7, R38, R86, R87, R88

Commit message: almost done
Parts:
- removed C22, C23, C24, C25, C27, C28: 100n, omat_ic_2:CAP0603
- added H4: GRN, omat_ic_2:LEDCHIP-LED0603
- added R54: 499, omat_ic_2:RES0603
Connections:
- new net N$17: H4.C, R54.2
- net +3V3: now also H4.A; no longer C22.1, C23.1, C24.1, C25.1, C27.1, C28.1
- net GND: now also R54.1; no longer C22.2, C23.2, C24.2, C25.2, C27.2, C28.2
Other:
- moved on the sheet: C26
Changed lines of the file:
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@@
 <part name="C21" library="omat_ic_2" deviceset="CAP" device="0603" value="2u2"/>
 <part name="GND48" library="EKE" deviceset="GND" device=""/>
-<part name="C22" library="omat_ic_2" deviceset="CAP" device="0603" value="100n"/>
-<part name="GND49" library="EKE" deviceset="GND" device=""/>
-<part name="+3V9" library="EKE" deviceset="+3V3" device=""/>
-<part name="C23" library="omat_ic_2" deviceset="CAP" device="0603" value="100n"/>
-<part name="GND50" library="EKE" deviceset="GND" device=""/>
-<part name="+3V10" library="EKE" deviceset="+3V3" device=""/>
-<part name="C24" library="omat_ic_2" deviceset="CAP" device="0603" value="100n"/>
-<part name="GND51" library="EKE" deviceset="GND" device=""/>
-<part name="+3V11" library="EKE" deviceset="+3V3" device=""/>
-<part name="C25" library="omat_ic_2" deviceset="CAP" device="0603" value="100n"/>
-<part name="GND52" library="EKE" deviceset="GND" device=""/>
-<part name="+3V12" library="EKE" deviceset="+3V3" device=""/>
 <part name="C26" library="omat_ic_2" deviceset="CAP" device="0603" value="100n"/>
 <part name="GND53" library="EKE" deviceset="GND" device=""/>
 <part name="+3V13" library="EKE" deviceset="+3V3" device=""/>
-<part name="C27" library="omat_ic_2" deviceset="CAP" device="0603" value="100n"/>
-<part name="GND54" library="EKE" deviceset="GND" device=""/>
-<part name="+3V14" library="EKE" deviceset="+3V3" device=""/>
-<part name="C28" library="omat_ic_2" deviceset="CAP" device="0603" value="100n"/>
-<part name="GND55" library="EKE" deviceset="GND" device=""/>
-<part name="+3V15" library="EKE" deviceset="+3V3" device=""/>
 <part name="C29" library="omat_ic_2" deviceset="CAP" device="0603" value="100n"/>
 <part name="GND56" library="EKE" deviceset="GND" device=""/>
@@
 <part name="V5" library="lippa" deviceset="SMAJXXA" device=""/>
 <part name="GND87" library="lippa" deviceset="GND" device=""/>
+<part name="H4" library="omat_ic_2" deviceset="LED" device="CHIP-LED0603" value="GRN"/>
+<part name="R54" library="omat_ic_2" deviceset="RES" device="0603" value="499"/>
+<part name="+3V9" library="lippa" deviceset="+3V3" device=""/>
 </parts>
 <sheets>
@@
 <attribute name="VALUE" x="233.68" y="38.1" size="1.778" layer="96"/>
 </instance>
-<instance part="C22" gate="G$1" x="292.1" y="175.26" smashed="yes">
-<attribute name="NAME" x="293.624" y="175.641" size="1.778" layer="95"/>
-<attribute name="VALUE" x="293.624" y="170.561" size="1.778" layer="96"/>
-</instance>
-<instance part="GND49" gate="1" x="292.1" y="167.64" smashed="yes">
-<attribute name="VALUE" x="289.56" y="165.1" size="1.778" layer="96"/>
-</instance>
-<instance part="+3V9" gate="G$1" x="292.1" y="180.34" smashed="yes">
-<attribute name="VALUE" x="289.56" y="175.26" size="1.778" layer="96" rot="R90"/>
-</instance>
-<instance part="C23" gate="G$1" x="302.26" y="175.26" smashed="yes">
-<attribute name="NAME" x="303.784" y="175.641" size="1.778" layer="95"/>
-<attribute name="VALUE" x="303.784" y="170.561" size="1.778" layer="96"/>
-</instance>
-<instance part="GND50" gate="1" x="302.26" y="167.64" smashed="yes">
-<attribute name="VALUE" x="299.72" y="165.1" size="1.778" layer="96"/>
-</instance>
-<instance part="+3V10" gate="G$1" x="302.26" y="180.34" smashed="yes">
-<attribute name="VALUE" x="299.72" y="175.26" size="1.778" layer="96" rot="R90"/>
-</instance>
-<instance part="C24" gate="G$1" x="312.42" y="175.26" smashed="yes">
-<attribute name="NAME" x="313.944" y="175.641" size="1.778" layer="95"/>
-<attribute name="VALUE" x="313.944" y="170.561" size="1.778" layer="96"/>
-</instance>
-<instance part="GND51" gate="1" x="312.42" y="167.64" smashed="yes">
-<attribute name="VALUE" x="309.88" y="165.1" size="1.778" layer="96"/>
-</instance>
-<instance part="+3V11" gate="G$1" x="312.42" y="180.34" smashed="yes">
-<attribute name="VALUE" x="309.88" y="175.26" size="1.778" layer="96" rot="R90"/>
-</instance>
-<instance part="C25" gate="G$1" x="322.58" y="175.26" smashed="yes">
-<attribute name="NAME" x="324.104" y="175.641" size="1.778" layer="95"/>
-<attribute name="VALUE" x="324.104" y="170.561" size="1.778" layer="96"/>
-</instance>
-<instance part="GND52" gate="1" x="322.58" y="167.64" smashed="yes">
-<attribute name="VALUE" x="320.04" y="165.1" size="1.778" layer="96"/>
-</instance>
-<instance part="+3V12" gate="G$1" x="322.58" y="180.34" smashed="yes">
-<attribute name="VALUE" x="320.04" y="175.26" size="1.778" layer="96" rot="R90"/>
-</instance>
-<instance part="C26" gate="G$1" x="332.74" y="175.26" smashed="yes">
-<attribute name="NAME" x="334.264" y="175.641" size="1.778" layer="95"/>
-<attribute name="VALUE" x="334.264" y="170.561" size="1.778" layer="96"/>
-</instance>
-<instance part="GND53" gate="1" x="332.74" y="167.64" smashed="yes">
-<attribute name="VALUE" x="330.2" y="165.1" size="1.778" layer="96"/>
-</instance>
-<instance part="+3V13" gate="G$1" x="332.74" y="180.34" smashed="yes">
-<attribute name="VALUE" x="330.2" y="175.26" size="1.778" layer="96" rot="R90"/>
-</instance>
-<instance part="C27" gate="G$1" x="292.1" y="157.48" smashed="yes">
-<attribute name="NAME" x="293.624" y="157.861" size="1.778" layer="95"/>
-<attribute name="VALUE" x="293.624" y="152.781" size="1.778" layer="96"/>
-</instance>
-<instance part="GND54" gate="1" x="292.1" y="149.86" smashed="yes">
-<attribute name="VALUE" x="289.56" y="147.32" size="1.778" layer="96"/>
-</instance>
-<instance part="+3V14" gate="G$1" x="292.1" y="162.56" smashed="yes">
-<attribute name="VALUE" x="289.56" y="157.48" size="1.778" layer="96" rot="R90"/>
-</instance>
-<instance part="C28" gate="G$1" x="302.26" y="157.48" smashed="yes">
+<instance part="C26" gate="G$1" x="302.26" y="157.48" smashed="yes">
 <attribute name="NAME" x="303.784" y="157.861" size="1.778" layer="95"/>
 <attribute name="VALUE" x="303.784" y="152.781" size="1.778" layer="96"/>
 </instance>
-<instance part="GND55" gate="1" x="302.26" y="149.86" smashed="yes">
+<instance part="GND53" gate="1" x="302.26" y="149.86" smashed="yes">
 <attribute name="VALUE" x="299.72" y="147.32" size="1.778" layer="96"/>
 </instance>
-<instance part="+3V15" gate="G$1" x="302.26" y="162.56" smashed="yes">
+<instance part="+3V13" gate="G$1" x="302.26" y="162.56" smashed="yes">
 <attribute name="VALUE" x="299.72" y="157.48" size="1.778" layer="96" rot="R90"/>
 </instance>
@@
 </segment>
 <segment>
-<pinref part="C22" gate="G$1" pin="2"/>
-<pinref part="GND49" gate="1" pin="GND"/>
-</segment>
-<segment>
-<pinref part="C23" gate="G$1" pin="2"/>
-<pinref part="GND50" gate="1" pin="GND"/>
-</segment>
-<segment>
-<pinref part="C24" gate="G$1" pin="2"/>
-<pinref part="GND51" gate="1" pin="GND"/>
-</segment>
-<segment>
-<pinref part="C25" gate="G$1" pin="2"/>
-<pinref part="GND52" gate="1" pin="GND"/>
-</segment>
-<segment>
 <pinref part="C26" gate="G$1" pin="2"/>
 <pinref part="GND53" gate="1" pin="GND"/>
 </segment>
 <segment>
-<pinref part="C27" gate="G$1" pin="2"/>
-<pinref part="GND54" gate="1" pin="GND"/>
-</segment>
-<segment>
-<pinref part="C28" gate="G$1" pin="2"/>
-<pinref part="GND55" gate="1" pin="GND"/>
-</segment>
-<segment>
 <pinref part="C29" gate="G$1" pin="2"/>
 <pinref part="GND56" gate="1" pin="GND"/>
@@
 </segment>
 <segment>
-<pinref part="C22" gate="G$1" pin="1"/>
-<pinref part="+3V9" gate="G$1" pin="+3V3"/>
-</segment>
-<segment>
-<pinref part="C23" gate="G$1" pin="1"/>
-<pinref part="+3V10" gate="G$1" pin="+3V3"/>
-</segment>
-<segment>
-<pinref part="C24" gate="G$1" pin="1"/>
-<pinref part="+3V11" gate="G$1" pin="+3V3"/>
-</segment>
-<segment>
-<pinref part="C25" gate="G$1" pin="1"/>
-<pinref part="+3V12" gate="G$1" pin="+3V3"/>
-</segment>
-<segment>
 <pinref part="C26" gate="G$1" pin="1"/>
 <pinref part="+3V13" gate="G$1" pin="+3V3"/>
 </segment>
 <segment>
-<pinref part="C27" gate="G$1" pin="1"/>
-<pinref part="+3V14" gate="G$1" pin="+3V3"/>
-</segment>
-<segment>
-<pinref part="C28" gate="G$1" pin="1"/>
-<pinref part="+3V15" gate="G$1" pin="+3V3"/>
-</segment>
-<segment>
 <pinref part="C29" gate="G$1" pin="1"/>
 <pinref part="+3V16" gate="G$1" pin="+3V3"/>
@@
 <attribute name="VALUE" x="90.17" y="34.798" size="1.778" layer="96"/>
 </instance>
+<instance part="H4" gate="G$1" x="266.7" y="248.92" smashed="yes" rot="R90">
+<attribute name="NAME" x="271.272" y="252.476" size="1.778" layer="95" rot="R180"/>
+<attribute name="VALUE" x="266.192" y="252.476" size="1.778" layer="96" rot="R180"/>
+</instance>
+<instance part="R54" gate="G$1" x="279.4" y="248.92" smashed="yes" rot="R180">
+<attribute name="NAME" x="283.21" y="247.4214" size="1.778" layer="95" rot="R180"/>
+<attribute name="VALUE" x="283.21" y="252.222" size="1.778" layer="96" rot="R180"/>
+</instance>
+<instance part="+3V9" gate="G$1" x="251.46" y="256.54" smashed="yes">
+<attribute name="VALUE" x="251.46" y="259.08" size="1.778" layer="96" align="top-center"/>
+</instance>
 </instances>
 <busses>
@@
 <wire x1="284.48" y1="228.6" x2="289.56" y2="228.6" width="0.1524" layer="91"/>
 <junction x="289.56" y="228.6"/>
+<pinref part="R54" gate="G$1" pin="1"/>
+<wire x1="284.48" y1="248.92" x2="289.56" y2="248.92" width="0.1524" layer="91"/>
+<wire x1="289.56" y1="248.92" x2="289.56" y2="238.76" width="0.1524" layer="91"/>
+<junction x="289.56" y="238.76"/>
 </segment>
 <segment>
@@
 <wire x1="175.26" y1="71.12" x2="175.26" y2="76.2" width="0.1524" layer="91"/>
 </segment>
+<segment>
+<pinref part="+3V9" gate="G$1" pin="+3V3"/>
+<wire x1="251.46" y1="254" x2="251.46" y2="248.92" width="0.1524" layer="91"/>
+<pinref part="H4" gate="G$1" pin="A"/>
+<wire x1="251.46" y1="248.92" x2="264.16" y2="248.92" width="0.1524" layer="91"/>
+</segment>
 </net>
 <net name="USART3TX" class="0">
@@
 </segment>
 </net>
+<net name="N$17" class="0">
+<segment>
+<pinref part="R54" gate="G$1" pin="2"/>
+<pinref part="H4" gate="G$1" pin="C"/>
+<wire x1="274.32" y1="248.92" x2="271.78" y2="248.92" width="0.1524" layer="91"/>
+</segment>
+</net>
