File: lippa.sch (EAGLE design)
At the start: 149 parts, among them K1 629105136821, X1 B4B-PH-K-S, X10 PIIKKIRIMA-3, X11 B8B-PH-K-S, X2 B4B-PH-K-S, X3 B4B-PH-K-S, X4 B4B-PH-K-S, X5 LIITTIMET_X3815-10, X7 PIIKKIRIMA-3, X8 B6B-PH-K-S, X9 PIIKKIRIMA-3, Y1 EKE_PTH3.2-6.5SQ, Y2 EKE_PTH3.2-6.5SQ, Y3 EKE_PTH3.2-6.5SQ, Y4 EKE_PTH3.2-6.5SQ

Commit message: Layout complete
Parts:
- added U$1: DAFUG, lippa:DAFUG
- renumbered K1 to X12
Connections:
- net N$14 renamed SERVO_2
- net N$15 renamed SERVO_1
- net N$16 renamed SERVO_3
Changed lines of the file:
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@@
 <part name="V1" library="cpu" deviceset="2N3904" device=""/>
 <part name="R37" library="aux-io" deviceset="PASSIIVIT_RES" device="0603" value="1k47"/>
-<part name="K1" library="cpu" deviceset="629105136821" device=""/>
+<part name="X12" library="cpu" deviceset="629105136821" device=""/>
 <part name="GND45" library="EKE" deviceset="GND" device=""/>
 <part name="+3V21" library="cpu" deviceset="+3V3" device=""/>
@@
 <part name="R54" library="omat_ic_2" deviceset="RES" device="0603" value="499"/>
 <part name="+3V9" library="lippa" deviceset="+3V3" device=""/>
+<part name="U$1" library="lippa" deviceset="DAFUG" device=""/>
+<part name="U$2" library="lippa" deviceset="OSHW" device=""/>
 </parts>
 <sheets>
@@
 <attribute name="VALUE" x="99.06" y="106.68" size="1.778" layer="96"/>
 </instance>
+<instance part="U$1" gate="G$1" x="312.42" y="30.48" smashed="yes"/>
+<instance part="U$2" gate="G$1" x="347.98" y="40.64" smashed="yes"/>
 </instances>
 <busses>
@@
 </segment>
 </net>
-<net name="N$14" class="0">
+<net name="SERVO_2" class="0">
 <segment>
 <pinref part="X9" gate="G$1" pin="1"/>
@@
 <wire x1="287.02" y1="180.34" x2="279.4" y2="180.34" width="0.1524" layer="91"/>
 <pinref part="R41" gate="G$1" pin="2"/>
+<label x="314.96" y="170.18" size="1.778" layer="95"/>
 </segment>
 </net>
-<net name="N$15" class="0">
+<net name="SERVO_1" class="0">
 <segment>
 <pinref part="X7" gate="G$1" pin="1"/>
 <wire x1="279.4" y1="187.96" x2="337.82" y2="187.96" width="0.1524" layer="91"/>
 <pinref part="R40" gate="G$1" pin="2"/>
+<label x="317.5" y="187.96" size="1.778" layer="95"/>
 </segment>
 </net>
-<net name="N$16" class="0">
+<net name="SERVO_3" class="0">
 <segment>
 <pinref part="X10" gate="G$1" pin="1"/>
@@
 <wire x1="281.94" y1="172.72" x2="279.4" y2="172.72" width="0.1524" layer="91"/>
 <pinref part="R42" gate="G$1" pin="2"/>
+<label x="314.96" y="152.4" size="1.778" layer="95"/>
 </segment>
 </net>
@@
 <attribute name="VALUE" x="66.802" y="113.03" size="1.778" layer="96" rot="R90"/>
 </instance>
-<instance part="K1" gate="G$1" x="27.94" y="167.64" smashed="yes" rot="MR0">
+<instance part="X12" gate="G$1" x="27.94" y="167.64" smashed="yes" rot="MR0">
 <attribute name="NAME" x="35.56" y="181.61" size="1.778" layer="95" rot="MR0"/>
 <attribute name="VALUE" x="35.56" y="162.56" size="1.778" layer="96" rot="MR0"/>
@@
 </segment>
 <segment>
-<pinref part="K1" gate="G$1" pin="5"/>
+<pinref part="X12" gate="G$1" pin="5"/>
 <wire x1="38.1" y1="167.64" x2="43.18" y2="167.64" width="0.1524" layer="91"/>
 <pinref part="GND45" gate="1" pin="GND"/>
@@
 <label x="50.8" y="175.26" size="1.778" layer="95"/>
 <wire x1="127" y1="175.26" x2="38.1" y2="175.26" width="0.1524" layer="91"/>
-<pinref part="K1" gate="G$1" pin="2"/>
+<pinref part="X12" gate="G$1" pin="2"/>
 <pinref part="D2" gate="G$2" pin="PA11"/>
 </segment>
@@
 <wire x1="48.26" y1="172.72" x2="38.1" y2="172.72" width="0.1524" layer="91"/>
 <junction x="48.26" y="172.72"/>
-<pinref part="K1" gate="G$1" pin="3"/>
+<pinref part="X12" gate="G$1" pin="3"/>
 <pinref part="D2" gate="G$2" pin="PA12"/>
 </segment>
@@
 <wire x1="76.2" y1="177.8" x2="38.1" y2="177.8" width="0.1524" layer="91"/>
 <label x="50.8" y="177.8" size="1.778" layer="95"/>
-<pinref part="K1" gate="G$1" pin="1"/>
+<pinref part="X12" gate="G$1" pin="1"/>
 <pinref part="V26" gate="G$1" pin="VCC"/>
 <wire x1="68.58" y1="220.98" x2="76.2" y2="220.98" width="0.1524" layer="91"/>
